Commit message: Some URDF changes for the XMaxx

File: urdf/_materials.xacro (robot description, xacro)
@@ -5,4 +5,7 @@
   <material name="LightBlue">
     <color rgba="0.4 0.4 1.0 1.0" />
+  </material>
+  <material name="LightGreen">
+    <color rgba="0.2 1.0 0.0 1.0" />
   </material>
   <material name="White">

File: urdf/_rc_parts.xacro (robot description, xacro)
@@ -10,4 +10,7 @@
     wheel_width
     wheel_radius
+    wheel_base
+    spur_width
+    chassis_clearance
    -->
   <xacro:macro name="wheel" params="prefix suffix reflect mirror">
@@ -22,4 +25,5 @@
       </visual>
       <collision>
+        <origin xyz="0 0 0" rpy="0 ${pi/2} 0" />
         <geometry>
           <cylinder length="${wheel_width}" radius="${wheel_radius}" />
@@ -30,5 +34,5 @@
       <parent link="base_link" />
       <child link="${prefix}_${suffix}_wheel_link" />
-      <origin xyz="${wheel_base/2*mirror}  ${0.1015*reflect} 0.030" rpy="0 0 ${(pi/2)*reflect}" />
+      <origin xyz="${wheel_base/2*mirror}  ${spur_width*reflect} ${wheel_radius-chassis_clearance}" rpy="0 0 ${(pi/2)*reflect}" />
     </joint>
   </xacro:macro>

File: urdf/xmaxx.xacro (robot description, xacro)
@@ -1,5 +1,5 @@
 <?xml version="1.0" encoding="UTF-8" ?>
 <robot
-  name="stampede"
+  name="xmaxx"
   xmlns:xacro="http://www.ros.org/wiki/xacro">
   <!--  -->
@@ -8,13 +8,13 @@
   <xacro:include filename="$(find robo_magellan)/urdf/_rc_parts.xacro" />
   <!-- Parameterized robot dimensions -->
-  <xacro:property name="wheel_radius" value="0.060" />
-  <xacro:property name="wheel_width" value="0.065" />
-  <xacro:property name="wheel_base" value="0.270" />
-  <xacro:property name="spur_width" value="0.1015" />
-  <xacro:property name="chassis_width" value="0.270" />
-  <xacro:property name="chassis_length" value="0.380" />
-  <xacro:property name="chassis_height" value="0.160" />
+  <xacro:property name="wheel_radius" value="0.104" />
+  <xacro:property name="wheel_width" value="0.110" />
+  <xacro:property name="wheel_base" value="0.485" />
+  <xacro:property name="spur_width" value="0.225" />
+  <xacro:property name="chassis_width" value="0.325" />
+  <xacro:property name="chassis_length" value="0.735" />
+  <xacro:property name="chassis_height" value="0.250" />
   <xacro:property name="chassis_clearance" value="0.120" />
-  <xacro:property name="chassis_mass" value="1.85" />
+  <xacro:property name="chassis_mass" value="5.85" />
   <link name="base_link">
     <visual>
@@ -65,15 +65,15 @@
   </joint>
   <link name="_base_link">
-    <visual>
-      <origin xyz="0 0 0" rpy="0 0 0" />
-      <geometry>
-        <box size="0.05 0.05 0.001" />
-      </geometry>
-      <material name="LightGreen" />
-    </visual>
+      <visual>
+        <origin xyz="0 0 0" rpy="0 0 0" />
+        <geometry>
+          <box size="0.5 0.5 0.001" />
+        </geometry>
+        <material name="LightGreen" />
+      </visual>
     <collision>
       <geometry>
-        <box size="0.05 0.05 0.001" />
-      </geometry>
+          <box size="0.5 0.5 0.001" />
+        </geometry>
     </collision>
   </link>
